File: pcb/multi-midi/multi-midi.kicad_pcb (KiCad board)
At the start: 2 copper layers, 101.2 x 71.1 mm, 60 parts, among them J1 DIN-5_180degree, J10 Conn_01x04_Male, J11 Conn_01x04_Male, J12 Barrel_Jack_Switch, J13 Conn_01x03_Male, J2 DIN-5_180degree, J3 DIN-5_180degree, J4 DIN-5_180degree, J5 DIN-5_180degree, J6 DIN-5_180degree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

Commit message: Swap out inductors with a "basic part"
Version of how I ordered rev0.
Parts:
- L1, L10, L11, L12, L13, L14, L15, L16, L17, L2, L3, L4, L5, L6, L7, L8, L9: value SZ1608K102TF -> SDFL2012S100KTF; footprint Inductor_SMD:L_0603_1608Metric -> Inductor_SMD:L_0805_2012Metric
- L18: value SZ1608K102TF -> SDFL2012S100KTF; footprint Resistor_SMD:R_0603_1608Metric -> Inductor_SMD:L_0805_2012Metric
- moved L18 0.25 mm to (112.9, 93.7)
- moved L17 0.13 mm to (112.9, 97.5)
Routing:
- net /BUFFER_C: track 31.5 -> 32.9 mm
Other:
- board text added: "JLCJLCJLCJLC"
- board text added: "Mfr. Order No.:"
